File: boards/pcb/hyperpotato.kicad_sch (KiCad schematic)
At the start: 85 parts, among them J1 HRO_TYPE-C-31-M-14, J2 T460S Module, J3 Battery, J5 Conn_01x04_Socket, M1 Motor_DC, Q1 2N7002, Q2 AO3401A, Q3 AO3401A, SW1 SW_Push_45deg, SW10 SW_Push_45deg, SW11 SW_Push_45deg, SW12 SW_Push_45deg, SW13 SW_Push_45deg, SW14 SW_Push_45deg, SW15 PWR, SW16 RST, SW2 SW_Push_45deg, SW3 SW_Push_45deg, SW4 SW_Push_45deg, SW5 SW_Push_45deg, SW6 SW_Push_45deg, SW7 SW_Push_45deg, SW8 SW_Push_45deg, SW9 SW_Push_45deg, U1 DRV2605LDGS, U2 SRV05-4, U3 BQ24075, U4 MAX17048, U5 nRF52840_E73-2G4M08S1C, U6 T460S, Y1 32.768 KHz

Commit message: Add schematic labels on mcu
Connections:
- net +BATT: now also R12.1; no longer R12.2
- net SCL: no longer U5.15 (P0.05/AIN3)
- net SDA: no longer U5.22 (P0.07)
- net at SW15.1 (A): now also R12.2; no longer R12.1
- net P1.11: now reaches U5.1 (P1.11)
- net P0.26: now reaches U5.12 (P0.26)
- net P0.06: now reaches U5.14 (P0.06)
- net P0.08: now reaches U5.16 (P0.08)
- net P1.09: now reaches U5.17 (P1.09)
- net P0.04: now reaches U5.18 (P0.04/AIN2)
- net P.1.10: now reaches U5.2 (P1.10)
- net P0.12: now reaches U5.20 (P0.12)
- net P0.15: now reaches U5.28 (P0.15)
- net P0.03: now reaches U5.3 (P0.03/AIN1)
- net P0.17: now reaches U5.30 (P0.17)
- net P0.20: now reaches U5.32 (P0.20)
- net P0.13: now reaches U5.33 (P0.13)
- net P0.24: now reaches U5.35 (P0.24)
- net P1.02: now reaches U5.38 (P1.02)
- net P1.04: now reaches U5.40 (P1.04)
- net P0.09: now reaches U5.41 (P0.09/NFC1)
- net P1.06: now reaches U5.42 (P1.06)
- net P0.10: now reaches U5.43 (P0.10/NFC2)
- net P1.13: now reaches U5.6 (P1.13)
- net P0.31: now reaches U5.9 (P0.31/AIN7)
- net UG_EN renamed P1.00
- net UG_LV renamed P0.22
- net col0 renamed P0.02
- net col1 renamed P0.28
- net row0 renamed P0.29
- net row1 renamed P0.30
- new net P0.05: U5.15 (P0.05/AIN3)
- new net P0.07: U5.22 (P0.07)
Other:
- moved on the sheet: D1, D10, D11, D12, D13, D14, D2, D3, D4, D5, D6, D7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
