File: pcb/hyperpotato.kicad_pcb (KiCad board)
At the start: 2 copper layers, 117 x 88.3 mm, 46 parts, among them J1 Conn_01x02_Socket, J2 Conn_01x03_Pin, Q1 AO3401A, SW1 SW_Push_45deg, SW10 SW_Push_45deg, SW11 SW_Push_45deg, SW12 SW_Push_45deg, SW13 SW_Push_45deg, SW14 SW_SPDT, SW15 SW_Push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

Commit message: Almost done!
Parts:
- added H2: MountingHole, hyperpotato:MountingHole, F.Cu at (148.2, 101.7)
- added H3: MountingHole, hyperpotato:MountingHole, F.Cu at (172.5, 155.5)
- added H4: MountingHole, hyperpotato:MountingHole, F.Cu at (187.5, 86.4)
- added H5: MountingHole, hyperpotato:MountingHole, F.Cu at (198.3, 129.0)
- added H6: MountingHole, hyperpotato:MountingHole, F.Cu at (216.2, 78.2)
- added H7: MountingHole, hyperpotato:MountingHole, F.Cu at (247.8, 141.3)
- C1, C2: footprint ssbb_parts_reversible:C_1206_3216Metric_reversible -> hyperpotato:C_1206_3216Metric_reversible
- D1, D10, D11, D12, D13, D2, D3, D4, D5, D6, D7, D8, D9: footprint ssbb_parts_reversible:D_1206_3216Metric_reversible -> hyperpotato:D_1206_3216Metric_reversible
- H1: footprint ssbb_parts:TP_Lenovo_T460S_Sensor -> hyperpotato:TP_Lenovo_T460S_Sensor
- J1: footprint ssbb_parts_reversible:Molex_Pico-EZmate_78171-0002_1x02-1MP_P1.20mm_Vertical_reversible -> hyperpotato:Molex_Pico-EZmate_78171-0002_1x02-1MP_P1.20mm_Vertical_reversible
- J2: footprint ssbb_parts:ELV1411A_reversible -> hyperpotato:ELV1411A_reversible
- R1, R2, R3, R4: footprint ssbb_parts_reversible:R_1206_3216Metric_reversible -> hyperpotato:R_1206_3216Metric_reversible
- SW14: footprint ssbb_parts_reversible:SW_SPDT_PCM12_reversible -> hyperpotato:SW_SPDT_PCM12_reversible
- SW15: footprint ssbb_parts:SW_SPST_SKQG_WithStem_reversible -> hyperpotato:Panasonic_EVQPUL_EVQPUC_reversible
- U1: footprint hyperpotato:XIAO-nRF52840-Sense-14P-2.54-21X17.8MM_reversible -> hyperpotato:Seed_Studio_XIAO_nRF52840_reversible
- U2: footprint ssbb_parts:TP_Sensor_Connector_reversible -> hyperpotato:TP_Sensor_Connector_reversible
- U3: footprint ssbb_parts:TP_Sprintek_SK8707-01_reversible -> hyperpotato:TP_Sprintek_SK8707-01_reversible
- U4: footprint ssbb_parts_reversible:VSSOP-10_3x3mm_P0.5mm_reversible -> hyperpotato:VSSOP-10_3x3mm_P0.5mm_reversible
- U5: footprint ssbb_parts_reversible:TSSOP-16_4.4x5mm_P0.65mm_reversible -> hyperpotato:TSSOP-16_4.4x5mm_P0.65mm_reversible
- moved SW15 41.5 mm to (171.2, 78.0), turned to 5 degrees
- moved SW14 9.91 mm to (179.7, 77.2)
- moved D15 9.04 mm to (234.8, 81.2)
- moved Q1 9.04 mm to (157.7, 110.4)
- moved SW2 9.04 mm to (198.3, 83.9)
- moved U1 9.04 mm to (156.4, 88.1)
- moved D4 9.04 mm to (247.4, 96.6)
- moved R2 9.04 mm to (227.0, 81.2)
- moved R1 9.04 mm to (157.7, 114.6)
- moved D2 9.04 mm to (247.4, 109.6)
- moved D8 9.04 mm to (250.5, 103.1)
- moved SW7 9.04 mm to (198.3, 100.9)
- moved SW9 9.04 mm to (234.3, 116.3)
- moved R3 9.04 mm to (230.9, 85.1)
- moved C2 9.04 mm to (152.0, 110.4)
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Connections:
- net +3.3V_OPTIONAL renamed +3.3V_TP
- U2 pad 1: TP_S1 -> TP_VCC
- U2 pad 2: TP_S2 -> TP_GND
- U2 pad 3: TP_S3 -> TP_Y
- U2 pad 4: TP_S4 -> TP_X
Routing:
- net TP_S1: track 93.1 -> 0.00 mm, vias 2 -> 0
- net TP_VCC: track 0.00 -> 91.3 mm, vias 0 -> 2
- net TP_S4: track 88.6 -> 0.00 mm, vias 2 -> 0
- net TP_S2: track 86.4 -> 0.00 mm, vias 2 -> 0
- net TP_X: track 0.00 -> 86.1 mm, vias 0 -> 2
- net TP_S3: track 86.0 -> 0.00 mm, vias 2 -> 0
- net TP_Y: track 0.00 -> 83.7 mm, vias 0 -> 2
- net TP_GND: track 0.00 -> 81.9 mm, vias 0 -> 2
- net RESET: track 80.7 -> 36.0 mm
- net +BATT: track 32.3 -> 38.7 mm
- net VBAT: track 129.2 -> 123.3 mm
- net GND: track 31.2 -> 34.0 mm, vias 9 -> 14
- net Net-(J2-Pin_2): track 124.3 -> 121.9 mm
- net +3.3V_TP: track 61.9 -> 60.0 mm
- net Net-(J2-Pin_1): track 126.3 -> 124.6 mm
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Other:
- board text removed: "OFF"
- board text removed: "ON"
- board text removed: "RESET"

Commit message: Before breaking everything
Parts:
- removed H2, H5: MountingHole, hyperpotato:MountingHole
- moved H4 1.00 mm to (187.6, 87.4)
- moved H7 0.13 mm to (247.8, 141.4)
Changed lines of the file:
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@@
 		(pad_to_mask_clearance 0)
 		(allow_soldermask_bridges_in_footprints no)
-		(grid_origin 198.256603 117.926485)
+		(grid_origin 207.256603 126.426486)
 		(pcbplotparams
 			(layerselection 0x00010fc_ffffffff)
@@
 	(net 64 "unconnected-(U5-QH'-Pad9)_1")
 	(net 65 "unconnected-(SW14-C-Pad3)_1")
-	(footprint "hyperpotato:MountingHole"
-		(layer "F.Cu")
-		(at 148.156603 101.726485)
-		(descr "Mounting Hole 3.5mm")
-		(tags "mounting hole 3.5mm")
-		(property "Reference" "H2"
-			(at 0 -4.5 0)
-			(layer "F.SilkS")
-			(effects
-				(font
-					(size 1 1)
-					(thickness 0.15)
-				)
-			)
-		)
-		(property "Value" "MountingHole"
-			(at 0 4.5 0)
-			(layer "F.Fab")
-			(effects
-				(font
-					(size 1 1)
-					(thickness 0.15)
-				)
-			)
-		)
-		(property "Footprint" "hyperpotato:MountingHole"
-			(at 0 0 0)
-			(unlocked yes)
-			(layer "F.Fab")
-			(hide yes)
-			(effects
-				(font
-					(size 1.27 1.27)
-					(thickness 0.15)
-				)
-			)
-		)
-		(property "Datasheet" ""
-			(at 0 0 0)
-			(unlocked yes)
-			(layer "F.Fab")
-			(hide yes)
-			(effects
-				(font
-					(size 1.27 1.27)
-					(thickness 0.15)
-				)
-			)
-		)
-		(property "Description" "Mounting Hole without connection"
-			(at 0 0 0)
-			(unlocked yes)
-			(layer "F.Fab")
-			(hide yes)
-			(effects
-				(font
-					(size 1.27 1.27)
-					(thickness 0.15)
-				)
-			)
-		)
-		(property ki_fp_filters "MountingHole*")
-		(sheetname "Root")
-		(sheetfile "hyperpotato.kicad_sch")
-		(attr exclude_from_pos_files exclude_from_bom)
-		(fp_text user "${REFERENCE}"
-			(at 0 0 0)
-			(layer "F.Fab")
-			(effects
-				(font
-					(size 1 1)
-					(thickness 0.15)
-				)
-			)
-		)
-		(pad "1" thru_hole circle
-			(at 0 0)
-			(size 6.2 6.2)
-			(drill 3.6)
-			(layers "*.Cu" "*.Mask")
-			(remove_unused_layers no)
-		)
-	)
 	(footprint "hyperpotato:SW_Choc_Mini_reversible_1u"
 		(layer "F.Cu")
@@
 			(at 1.537497 2.068332 0)
 			(layer "F.SilkS")
+			(hide yes)
 			(effects
 				(font
@@
 			(at 0 2.4 90)
 			(layer "F.Fab")
+			(hide yes)
 			(effects
 				(font
@@
 			(at 0.000001 2.000001 135)
 			(layer "F.SilkS")
+			(hide yes)
 			(effects
 				(font
@@
 			(at 0 1.82 135)
 			(layer "F.Fab")
+			(hide yes)
 			(effects
 				(font
@@
 			(at 3.499996 0 90)
 			(layer "F.SilkS")
+			(hide yes)
 			(effects
 				(font
@@
 			(at 0 1.850001 90)
 			(layer "F.Fab")
+			(hide yes)
 			(effects
 				(font
@@
 			(at 3.318331 0.262503 0)
 			(layer "F.SilkS")
+			(hide yes)
 			(effects
 				(font
@@
 			(at 0 1.82 0)
 			(layer "F.Fab")
+			(hide yes)
 			(effects
 				(font
@@
 			(at 0.000001 2.000001 135)
 			(layer "F.SilkS")
+			(hide yes)
 			(effects
 				(font
@@
 			(at 0 1.82 135)
 			(layer "F.Fab")
+			(hide yes)
 			(effects
 				(font
@@
 		)
 	)
-	(footprint "hyperpotato:MountingHole"
-		(layer "F.Cu")
-		(at 198.256603 129.026485)
-		(descr "Mounting Hole 3.5mm")
-		(tags "mounting hole 3.5mm")
-		(property "Reference" "H5"
-			(at 0 -4.5 0)
-			(layer "F.SilkS")
-			(effects
-				(font
-					(size 1 1)
-					(thickness 0.15)
-				)
-			)
-		)
-		(property "Value" "MountingHole"
-			(at 0 4.5 0)
-			(layer "F.Fab")
-			(effects
-				(font
-					(size 1 1)
-					(thickness 0.15)
-				)
-			)
-		)
-		(property "Footprint" "hyperpotato:MountingHole"
-			(at 0 0 0)
-			(unlocked yes)
-			(layer "F.Fab")
-			(hide yes)
-			(effects
-				(font
-					(size 1.27 1.27)
-					(thickness 0.15)
-				)
-			)
-		)
-		(property "Datasheet" ""
-			(at 0 0 0)
-			(unlocked yes)
-			(layer "F.Fab")
-			(hide yes)
-			(effects
-				(font
-					(size 1.27 1.27)
-					(thickness 0.15)
-				)
-			)
-		)
-		(property "Description" "Mounting Hole without connection"
-			(at 0 0 0)
-			(unlocked yes)
-			(layer "F.Fab")
-			(hide yes)
-			(effects
-				(font
-					(size 1.27 1.27)
-					(thickness 0.15)
-				)
-			)
-		)
-		(property ki_fp_filters "MountingHole*")
-		(sheetname "Root")
-		(sheetfile "hyperpotato.kicad_sch")
-		(attr exclude_from_pos_files exclude_from_bom)
-		(fp_text user "${REFERENCE}"
-			(at 0 0 0)
-			(layer "F.Fab")
-			(effects
-				(font
-					(size 1 1)
-					(thickness 0.15)
-				)
-			)
-		)
-		(pad "1" thru_hole circle
-			(at 0 0)
-			(size 6.2 6.2)
-			(drill 3.6)
-			(layers "*.Cu" "*.Mask")
-			(remove_unused_layers no)
-		)
-	)
 	(footprint "hyperpotato:D_1206_3216Metric_reversible"
 		(layer "F.Cu")
@@
 			(at 0 -4.5 0)
 			(layer "F.SilkS")
+			(hide yes)
 			(effects
 				(font
@@
 			(at 0 4.5 0)
 			(layer "F.Fab")
+			(hide yes)
 			(effects
 				(font
@@
 	(footprint "hyperpotato:MountingHole"
 		(layer "F.Cu")
-		(at 187.456603 86.426485)
+		(at 187.556603 87.426485)
 		(descr "Mounting Hole 3.5mm")
 		(tags "mounting hole 3.5mm")
@@
 			(at 0 -4.5 0)
 			(layer "F.SilkS")
+			(hide yes)
 			(effects
 				(font
@@
 			(at 0 4.5 0)
 			(layer "F.Fab")
+			(hide yes)
 			(effects
 				(font
@@
 			(at 3.5 0 90)
 			(layer "F.SilkS")
+			(hide yes)
 			(effects
 				(font
@@
 			(at 0 1.850001 90)
 			(layer "F.Fab")
+			(hide yes)
 			(effects
 				(font
@@
 	(footprint "hyperpotato:MountingHole"
 		(layer "F.Cu")
-		(at 247.756602 141.296488)
+		(at 247.756602 141.426485)
 		(descr "Mounting Hole 3.5mm")
 		(tags "mounting hole 3.5mm")
@@
 			(at 0 -4.5 0)
 			(layer "F.SilkS")
+			(hide yes)
 			(effects
 				(font
@@
 			(at 0 4.5 0)
 			(layer "F.Fab")
+			(hide yes)
 			(effects
 				(font
@@
 			(at 0 -4 90)
 			(layer "F.SilkS")
+			(hide yes)
 			(effects
 				(font
@@
 			(at 0 3.449999 90)
 			(layer "F.Fab")
+			(hide yes)
 			(effects
 				(font
@@
 			(at 0 -4.5 0)
 			(layer "F.SilkS")
+			(hide yes)
 			(effects
 				(font
@@
 			(at 0 4.5 0)
 			(layer "F.Fab")
+			(hide yes)
 			(effects
 				(font
@@
 			(at 0 -2.591896 0)
 			(layer "F.SilkS")
+			(hide yes)
 			(effects
 				(font
@@
 			(at 0 2.450001 0)
 			(layer "F.Fab")
+			(hide yes)
 			(effects
 				(font
@@
 			(at 0 1.999998 135)
 			(layer "F.SilkS")
+			(hide yes)
 			(effects
 				(font
@@
 			(at 0 1.82 135)
 			(layer "F.Fab")
+			(hide yes)
 			(effects
 				(font

Commit message: Ready to go!
Parts:
- added H2: MountingHole, hyperpotato:MountingHole, F.Cu at (203.3, 129.4)
- moved SW13 5.49 mm to (252.8, 152.5)
- moved H5 5.10 mm to (252.8, 142.4)
- moved H3 5.09 mm to (177.5, 156.4)
- moved J1 5.06 mm to (236.0, 129.8)
- moved C2 5.01 mm to (157.0, 110.6)
- moved D1 5.01 mm to (258.6, 109.8)
- moved D16 5.01 mm to (243.8, 85.4)
- moved H1 5.01 mm to (230.3, 99.5)
- moved R3 5.01 mm to (235.9, 85.4)
- moved SW5 5.01 mm to (165.7, 125.5)
- moved SW9 5.01 mm to (239.3, 116.5)
- moved D3 5.01 mm to (258.6, 103.3)
- moved D6 5.01 mm to (252.4, 116.3)
- moved D7 5.01 mm to (255.5, 109.8)
- moved H6 5.01 mm to (221.2, 78.4)
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- renumbered H7 to H5
Routing:
- net Net-(D13-A): track 39.5 -> 41.9 mm
- net COL4: track 191.2 -> 193.6 mm
- net TP_GND: track 81.9 -> 84.0 mm
- net TP_DATA: track 113.2 -> 111.9 mm
- net TP_CLK: track 107.4 -> 106.5 mm
- net GND: vias 14 -> 13
Other:
- board size 117 x 88.3 mm -> 117 x 90.3 mm
