File: pcb/hyperpotato.kicad_sch (KiCad schematic)
At the start: 46 parts, among them J1 Conn_01x02_Socket, J2 Conn_01x03_Pin, Q1 AO3401A, SW1 SW_Push_45deg, SW10 SW_Push_45deg, SW11 SW_Push_45deg, SW12 SW_Push_45deg, SW13 SW_Push_45deg, SW14 SW_SPDT, SW15 SW_Push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

Commit message: Use in-house footprints,
Parts:
- C1, C2: footprint ssbb_parts_reversible:C_1206_3216Metric_reversible -> hyperpotato:C_1206_3216Metric_reversible
- D1, D10, D11, D12, D13, D2, D3, D4, D5, D6, D7, D8, D9: footprint ssbb_parts_reversible:D_1206_3216Metric_reversible -> hyperpotato:D_1206_3216Metric_reversible
- H1: value MountingHole -> T460S; footprint ssbb_parts:TP_Lenovo_T460S_Sensor -> hyperpotato:TP_Lenovo_T460S_Sensor
- J1: footprint ssbb_parts_reversible:Molex_Pico-EZmate_78171-0002_1x02-1MP_P1.20mm_Vertical_reversible -> hyperpotato:Molex_Pico-EZmate_78171-0002_1x02-1MP_P1.20mm_Vertical_reversible
- J2: footprint ssbb_parts:ELV1411A_reversible -> hyperpotato:ELV1411A_reversible
- R1: footprint ssbb_parts_reversible:R_1206_3216Metric_reversible -> hyperpotato:R_1206_3216Metric_reversible
- R2: renamed from R6; footprint ssbb_parts_reversible:R_1206_3216Metric_reversible -> hyperpotato:R_1206_3216Metric_reversible
- R3: renamed from R7; footprint ssbb_parts_reversible:R_1206_3216Metric_reversible -> hyperpotato:R_1206_3216Metric_reversible
- R4: renamed from R8; footprint ssbb_parts_reversible:R_1206_3216Metric_reversible -> hyperpotato:R_1206_3216Metric_reversible
- SW14: footprint ssbb_parts_reversible:SW_SPDT_PCM12_reversible -> hyperpotato:SW_SPDT_PCM12_reversible
- SW15: footprint ssbb_parts:SW_SPST_SKQG_WithStem_reversible -> hyperpotato:Panasonic_EVQPUL_EVQPUC_reversible
- U1: footprint hyperpotato:XIAO-nRF52840-Sense-14P-2.54-21X17.8MM_1 -> hyperpotato:Seed_Studio_XIAO_nRF52840_reversible
- U2: footprint ssbb_parts:TP_Sensor_Connector_reversible -> hyperpotato:TP_Sensor_Connector_reversible; symbol ssbb_parts:Sprintek_SK8707-01_Sensor -> ssbb_parts:TP_Sprintek_SK8707-01_Sensor
- U3: footprint ssbb_parts:TP_Sprintek_SK8707-01_reversible -> hyperpotato:TP_Sprintek_SK8707-01_reversible; symbol ssbb_parts:Sprintek_SK8707–01 -> ssbb_parts:TP_Sprintek_SK8707–01
- U4: footprint ssbb_parts_reversible:VSSOP-10_3x3mm_P0.5mm_reversible -> hyperpotato:VSSOP-10_3x3mm_P0.5mm_reversible
- U5: footprint ssbb_parts_reversible:TSSOP-16_4.4x5mm_P0.65mm_reversible -> hyperpotato:TSSOP-16_4.4x5mm_P0.65mm_reversible
Connections:
- net SCL: now also U1.18 (P0.10-LF); no longer U1.17 (P0.09-LF)
- net SDA: now also U1.17 (P0.09-LF); no longer U1.18 (P0.10-LF)
- net TP_S1 renamed TP_VCC
- net TP_S2 renamed TP_GND
- net TP_S3 renamed TP_Y
- net TP_S4 renamed TP_X

Commit message: Almost done!
Parts:
- added H2, H3, H4, H5, H6, H7: MountingHole, hyperpotato:MountingHole, symbol Mechanical:MountingHole
Connections:
- net +3.3V_OPTIONAL renamed +3.3V_TP
- no-connect marks 8 -> 10

Commit message: Ready to go!
Parts:
- removed H7: MountingHole, hyperpotato:MountingHole, symbol Mechanical:MountingHole
Changed lines of the file:
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@@
-	)
-	(symbol
-		(lib_id "Mechanical:MountingHole")
-		(at 161.29 234.95 0)
-		(unit 1)
-		(exclude_from_sim yes)
-		(in_bom no)
-		(on_board yes)
-		(dnp no)
-		(fields_autoplaced yes)
-		(property "Reference" "H7"
-			(at 163.83 233.68 0)
-			(effects
-				(font
-					(size 1.27 1.27)
-				)
-				(justify left)
-			)
-		)
-		(property "Value" "MountingHole"
-			(at 163.83 236.22 0)
-			(effects
-				(font
-					(size 1.27 1.27)
-				)
-				(justify left)
-			)
-		)
-		(property "Footprint" "hyperpotato:MountingHole"
-			(at 161.29 234.95 0)
-			(effects
-				(font
-					(size 1.27 1.27)
-				)
-				(hide yes)
-			)
-		)
-		(property "Datasheet" "~"
-			(at 161.29 234.95 0)
-			(effects
-				(font
-					(size 1.27 1.27)
-				)
-				(hide yes)
-			)
-		)
-		(property "Description" "Mounting Hole without connection"
-			(at 161.29 234.95 0)
-			(effects
-				(font
-					(size 1.27 1.27)
-				)
-				(hide yes)
-			)
-		)
-		(instances
-			(project ""
-				(path "/19b5f7b9-14b9-4ffe-8621-f024a09d5ec4"
-					(reference "H7")
-					(unit 1)
-				)
-			)
-		)
 	)
 	(symbol
