File: pcb/pipra.kicad_sch (KiCad schematic)
At the start: 51 parts, among them J1 Conn_01x02_Socket, J2 Conn_01x03_Pin, Q1 AO3401A, SW1 SW_Push_45deg, SW10 SW_Push_45deg, SW11 SW_Push_45deg, SW12 SW_Push_45deg, SW13 SW_Push_45deg, SW14 SW_SPDT, SW15 SW_Push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

Commit message: After order
Connections:
- net +3.3V: no longer U4.5 (EN)
- net HAPTIC_EN: now reaches U1.4 (P0.29-D3-LF)
- net HAPTIC_EN: now also U4.5 (EN)
- no-connect marks 10 -> 9
Changed lines of the file:
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@@
 	)
 	(no_connect
-		(at 63.5 250.19)
-	)
-	(no_connect
 		(at 139.7 165.1)
 	)
@@
 	(wire
 		(pts
-			(xy 44.45 184.15) (xy 44.45 179.07)
+			(xy 33.02 180.34) (xy 33.02 179.07)
 		)
 		(stroke
@@
 	(wire
 		(pts
-			(xy 25.4 179.07) (xy 25.4 181.61)
-		)
-		(stroke
-			(width 0)
-			(type default)
-		)
-	)
-	(wire
-		(pts
 			(xy 100.33 237.49) (xy 100.33 247.65)
 		)
@@
 	(wire
 		(pts
-			(xy 25.4 181.61) (xy 45.72 181.61)
-		)
-		(stroke
-			(width 0)
-			(type default)
-		)
-	)
-	(wire
-		(pts
 			(xy 86.36 228.6) (xy 86.36 232.41)
 		)
@@
 	(wire
 		(pts
-			(xy 44.45 179.07) (xy 45.72 179.07)
+			(xy 33.02 179.07) (xy 45.72 179.07)
 		)
 		(stroke
@@
 		)
 	)
+	(global_label "HAPTIC_EN"
+		(shape input)
+		(at 45.72 181.61 180)
+		(fields_autoplaced yes)
+		(effects
+			(font
+				(size 1.27 1.27)
+			)
+			(justify right)
+		)
+		(property "Intersheetrefs" "${INTERSHEET_REFS}"
+			(at 34.9618 181.61 0)
+			(effects
+				(font
+					(size 1.27 1.27)
+				)
+				(justify right)
+				(hide yes)
+			)
+		)
+	)
 	(global_label "TP_X"
 		(shape input)
@@
 		)
 	)
+	(global_label "HAPTIC_EN"
+		(shape input)
+		(at 63.5 250.19 180)
+		(fields_autoplaced yes)
+		(effects
+			(font
+				(size 1.27 1.27)
+			)
+			(justify right)
+		)
+		(property "Intersheetrefs" "${INTERSHEET_REFS}"
+			(at 52.7418 250.19 0)
+			(effects
+				(font
+					(size 1.27 1.27)
+				)
+				(justify right)
+				(hide yes)
+			)
+		)
+	)
 	(global_label "ROW0"
 		(shape input)
@@
 	(symbol
 		(lib_id "power:GND")
-		(at 44.45 184.15 0)
+		(at 33.02 180.34 0)
 		(unit 1)
 		(exclude_from_sim no)
@@
 		(fields_autoplaced yes)
 		(property "Reference" "#PWR017"
-			(at 44.45 190.5 0)
+			(at 33.02 186.69 0)
 			(effects
 				(font
@@
 		)
 		(property "Value" "GND"
-			(at 44.45 189.23 0)
+			(at 33.02 185.42 0)
 			(effects
 				(font
@@
 		)
 		(property "Footprint" ""
-			(at 44.45 184.15 0)
+			(at 33.02 180.34 0)
 			(effects
 				(font
@@
 		)
 		(property "Datasheet" ""
-			(at 44.45 184.15 0)
+			(at 33.02 180.34 0)
 			(effects
 				(font
@@
 		)
 		(property "Description" "Power symbol creates a global label with name \"GND\" , ground"
-			(at 44.45 184.15 0)
+			(at 33.02 180.34 0)
 			(effects
 				(font
@@
 					(unit 1)
 				)
-			)
-		)
-	)
-	(symbol
-		(lib_id "power:+3.3V")
-		(at 25.4 179.07 0)
-		(unit 1)
-		(exclude_from_sim no)
-		(in_bom yes)
-		(on_board yes)
-		(dnp no)
-		(fields_autoplaced yes)
-		(property "Reference" "#PWR013"
-			(at 25.4 182.88 0)
-			(effects
-				(font
-					(size 1.27 1.27)
-				)
-				(hide yes)
-			)
-		)
-		(property "Value" "+3.3V"
-			(at 25.4 173.99 0)
-			(effects
-				(font
-					(size 1.27 1.27)
-				)
-			)
-		)
-		(property "Footprint" ""
-			(at 25.4 179.07 0)
-			(effects
-				(font
-					(size 1.27 1.27)
-				)
-				(hide yes)
-			)
-		)
-		(property "Datasheet" ""
-			(at 25.4 179.07 0)
-			(effects
-				(font
-					(size 1.27 1.27)
-				)
-				(hide yes)
-			)
-		)
-		(property "Description" "Power symbol creates a global label with name \"+3.3V\""
-			(at 25.4 179.07 0)
-			(effects
-				(font
-					(size 1.27 1.27)
-				)
-				(hide yes)
-			)
-		)
-		(pin "1"
-		)
-		(instances
-			(project ""
-				(path "/19b5f7b9-14b9-4ffe-8621-f024a09d5ec4"
-					(reference "#PWR013")
-					(unit 1)
-				)
