File: switch_plate/switch_plate.kicad_pcb (KiCad board)
At the start: 2 copper layers, 117 x 90.3 mm, 23 parts, among them SW1 SW_Push_45deg, SW10 SW_Push_45deg, SW11 SW_Push_45deg, SW12 SW_Push_45deg, SW13 SW_Push_45deg, SW2 SW_Push_45deg, SW3 SW_Push_45deg, SW4 SW_Push_45deg, SW5 SW_Push_45deg, SW6 SW_Push_45deg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

Commit message: After order
Parts:
- removed H7: Bottom Plate, pipra:BottomPlate
- moved H3 7.25 mm to (184.3, 157.6)
Changed lines of the file:
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@@
 			(drillshape 0)
 			(scaleselection 1)
-			(outputdirectory "pcb_gerbers")
+			(outputdirectory "switch_plate_gerbers")
 		)
 	)
@@
 		)
 		(fp_text user "CPG1232 - 12.7x13.7 plate cutout"
-			(at 0 -7.7 360)
+			(at 0 -7.7 0)
 			(layer "Cmts.User")
 			(effects
@@
 		)
 		(fp_text user "${VALUE}"
-			(at 0 8.254999 360)
+			(at 0 8.254999 0)
 			(layer "B.Fab")
 			(effects
@@
 		)
 		(fp_text user "CPG1232 - 12.7x13.7 plate cutout"
-			(at 0 -7.7 360)
+			(at 0 -7.7 0)
 			(layer "Cmts.User")
 			(effects
@@
 		)
 		(fp_text user "${VALUE}"
-			(at 0 8.254999 360)
+			(at 0 8.254999 0)
 			(layer "B.Fab")
 			(effects
@@
 		(at 254.401384 110.846253)
 		(property "Reference" "G***"
-			(at 0 0 360)
+			(at 0 0 0)
 			(layer "F.SilkS")
 			(hide yes)
@@
 		)
 		(property "Value" "LOGO"
-			(at 0.75 0 360)
+			(at 0.75 0 0)
 			(layer "F.SilkS")
 			(hide yes)
@@
 		)
 		(property "Footprint" "pipra:Graphics_Bamboo"
-			(at 0 0 360)
+			(at 0 0 0)
 			(layer "F.Fab")
 			(hide yes)
@@
 		)
 		(property "Datasheet" ""
-			(at 0 0 360)
+			(at 0 0 0)
 			(layer "F.Fab")
 			(hide yes)
@@
 		)
 		(property "Description" ""
-			(at 0 0 360)
+			(at 0 0 0)
 			(layer "F.Fab")
 			(hide yes)
@@
 		(at 175.893462 144.84142)
 		(property "Reference" "G***"
-			(at 0 0 360)
+			(at 0 0 0)
 			(layer "F.SilkS")
 			(hide yes)
@@
 		)
 		(property "Value" "LOGO"
-			(at 0.75 0 360)
+			(at 0.75 0 0)
 			(layer "F.SilkS")
 			(hide yes)
@@
 		)
 		(property "Footprint" "pipra:Graphics_Bird"
-			(at 0 0 360)
+			(at 0 0 0)
 			(layer "F.Fab")
 			(hide yes)
@@
 		)
 		(property "Datasheet" ""
-			(at 0 0 360)
+			(at 0 0 0)
 			(layer "F.Fab")
 			(hide yes)
@@
 		)
 		(property "Description" ""
-			(at 0 0 360)
+			(at 0 0 0)
 			(layer "F.Fab")
 			(hide yes)
@@
 		)
 		(fp_text user "CPG1232 - 12.7x13.7 plate cutout"
-			(at 0 -7.7 360)
+			(at 0 -7.7 0)
 			(layer "Cmts.User")
 			(effects
@@
 		)
 		(fp_text user "${VALUE}"
-			(at 0 8.254999 360)
+			(at 0 8.254999 0)
 			(layer "B.Fab")
 			(effects
@@
 		)
 		(fp_text user "CPG1232 - 12.7x13.7 plate cutout"
-			(at 0 -7.7 360)
+			(at 0 -7.7 0)
 			(layer "Cmts.User")
 			(effects
@@
 		)
 		(fp_text user "${VALUE}"
-			(at 0 8.254999 360)
+			(at 0 8.254999 0)
 			(layer "B.Fab")
 			(effects
@@
 		)
 		(fp_text user "CPG1232 - 12.7x13.7 plate cutout"
-			(at 0 -7.7 360)
+			(at 0 -7.7 0)
 			(layer "Cmts.User")
 			(effects
@@
 		)
 		(fp_text user "${VALUE}"
-			(at 0 8.254999 360)
+			(at 0 8.254999 0)
 			(layer "B.Fab")
 			(effects
@@
 	(footprint "MountingHole:MountingHole_2.2mm_M2_DIN965_Pad"
 		(layer "F.Cu")
-		(at 177.135195 156.452413)
+		(at 184.301195 157.572413)
 		(descr "Mounting Hole 2.2mm, M2, DIN965")
 		(tags "mounting hole 2.2mm m2 din965")
 		(property "Reference" "H3"
-			(at 0 -2.9 360)
+			(at 0 -2.9 0)
 			(layer "F.SilkS")
 			(hide yes)
@@
 		)
 		(property "Value" "MountingHole"
-			(at 0 2.9 360)
+			(at 0 2.9 0)
 			(layer "F.Fab")
 			(hide yes)
@@
 		)
 		(fp_text user "${REFERENCE}"
-			(at 0 0 360)
+			(at 0 0 0)
 			(layer "F.Fab")
 			(effects
@@
 		(tags "mounting hole 2.2mm m2 din965")
 		(property "Reference" "H4"
-			(at 0 -2.9 360)
+			(at 0 -2.9 0)
 			(layer "F.SilkS")
 			(hide yes)
@@
 		)
 		(property "Value" "MountingHole"
-			(at 0 2.9 360)
+			(at 0 2.9 0)
 			(layer "F.Fab")
 			(hide yes)
@@
 		)
 		(fp_text user "${REFERENCE}"
-			(at 0 0 360)
+			(at 0 0 0)
 			(layer "F.Fab")
 			(effects
@@
 		)
 		(fp_text user "CPG1232 - 12.7x13.7 plate cutout"
-			(at 0 -7.7 360)
+			(at 0 -7.7 0)
 			(layer "Cmts.User")
 			(effects
@@
 		)
 		(fp_text user "${VALUE}"
-			(at 0 8.254999 360)
+			(at 0 8.254999 0)
 			(layer "B.Fab")
 			(effects
@@
 		(tags "mounting hole 2.2mm m2 din965")
 		(property "Reference" "H5"
-			(at 0 -2.9 360)
+			(at 0 -2.9 0)
 			(layer "F.SilkS")
 			(hide yes)
@@
 		)
 		(property "Value" "MountingHole"
-			(at 0 2.9 360)
+			(at 0 2.9 0)
 			(layer "F.Fab")
 			(hide yes)
@@
 		)
 		(fp_text user "${REFERENCE}"
-			(at 0 0 360)
+			(at 0 0 0)
 			(layer "F.Fab")
 			(effects
@@
 		)
 	)
-	(footprint "pipra:BottomPlate"
-		(layer "F.Cu")
-		(at 108.701382 130.772404)
-		(property "Reference" "H7"
-			(at 0 -0.5 0)
-			(unlocked yes)
-			(layer "F.SilkS")
-			(hide yes)
-			(effects
-				(font
-					(size 1 1)
-					(thickness 0.1)
-				)
-			)
-		)
-		(property "Value" "Bottom Plate"
-			(at 0 1 0)
-			(unlocked yes)
-			(layer "F.Fab")
-			(hide yes)
-			(effects
-				(font
-					(size 1 1)
-					(thickness 0.15)
-				)
-			)
-		)
-		(property "Footprint" "pipra:BottomPlate"
-			(at 0 0 0)
-			(unlocked yes)
-			(layer "F.Fab")
-			(hide yes)
-			(effects
-				(font
-					(size 1 1)
-					(thickness 0.15)
-				)
-			)
-		)
-		(property "Datasheet" ""
-			(at 0 0 0)
-			(unlocked yes)
-			(layer "F.Fab")
-			(hide yes)
-			(effects
-				(font
-					(size 1 1)
-					(thickness 0.15)
-				)
-			)
-		)
-		(property "Description" "Mounting Hole without connection"
-			(at 0 0 0)
-			(unlocked yes)
-			(layer "F.Fab")
-			(hide yes)
-			(effects
-				(font
-					(size 1 1)
-					(thickness 0.15)
-				)
-			)
-		)
-		(property ki_fp_filters "MountingHole*")
-		(sheetname "Root")
-		(sheetfile "pipra.kicad_sch")
-		(attr smd exclude_from_bom)
-		(fp_text user "${REFERENCE}"
-			(at 0 2.5 0)
-			(unlocked yes)
-			(layer "F.Fab")
-			(effects
-				(font
-					(size 1 1)
-					(thickness 0.15)
-				)
-			)
-		)
-		(model "../3dmodels/bottom-plate.step"
-			(offset
-				(xyz 0 0 0)
-			)
-			(scale
-				(xyz 1 1 1)
-			)
-			(rotate
-				(xyz 0 0 0)
-			)
-		)
-	)
 	(footprint "pipra:SW_Choc_Mini_Plate_Cutout"
 		(layer "F.Cu")
@@
 		(tags "mounting hole 2.2mm m2 din965")
 		(property "Reference" "H6"
-			(at 0 -2.9 360)
+			(at 0 -2.9 0)
 			(layer "F.SilkS")
 			(hide yes)
@@
 		)
 		(property "Value" "MountingHole"
-			(at 0 2.9 360)
+			(at 0 2.9 0)
 			(layer "F.Fab")
 			(hide yes)
@@
 		)
 		(fp_text user "${REFERENCE}"
-			(at 0 0 360)
+			(at 0 0 0)
 			(layer "F.Fab")
 			(effects
@@
 		)
 		(fp_text user "CPG1232 - 12.7x13.7 plate cutout"
-			(at -1.553782 -7.564062 360)
+			(at -1.553782 -7.564062 0)
 			(layer "Cmts.User")
 			(effects
@@
 		)
 		(fp_text user "${VALUE}"
-			(at 0 8.254999 360)
+			(at 0 8.254999 0)
 			(layer "B.Fab")
 			(effects
@@
 		)
 		(fp_text user "CPG1232 - 12.7x13.7 plate cutout"
-			(at 0 -7.7 360)
+			(at 0 -7.7 0)
 			(layer "Cmts.User")
 			(effects
@@
 		)
 		(fp_text user "${VALUE}"
-			(at 0 8.254999 360)
+			(at 0 8.254999 0)
 			(layer "B.Fab")
 			(effects
@@
 		(tags "mounting hole 2.2mm m2 din965")
 		(property "Reference" "H2"
-			(at 0 -2.9 360)
+			(at 0 -2.9 0)
 			(layer "F.SilkS")
 			(hide yes)
@@
 		)
 		(property "Value" "MountingHole"
-			(at 0 2.9 360)
+			(at 0 2.9 0)
 			(layer "F.Fab")
 			(hide yes)
@@
 		)
 		(fp_text user "${REFERENCE}"
-			(at 0 0 360)
+			(at 0 0 0)
 			(layer "F.Fab")
 			(effects
